File: pcb/v1/eeprom-programmer.kicad_pcb (KiCad board)
At the start: 2 copper layers, 44.8 x 97 mm, 62 parts, among them J1 USB_C_Receptacle_USB2.0_16P, J2 Conn_01x04, J3 Conn_01x20, J4 Conn_01x20, SW1 SW_Push_Dual, SW2 SW_Push_Dual, SW3 SW_Push_Dual, U1 W25Q32JVSS, U2 USBLC6-2SC6, U3 RP2040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

Commit message: fix 2 mixed up labels; update output files; add pcb with rounded labels
Parts:
- moved C14 0.46 mm to (148.1, 67.5)
- moved R8 0.19 mm to (154.4, 77.8)
- moved C18 0.06 mm to (148.2, 72.0)
Routing:
- net +1V1: track 30.2 -> 34.4 mm
- net /RESET: track 50.2 -> 47.9 mm
- net /QSPI_SD0: track 14.3 -> 15.7 mm
- net /QSPI_SCLK: track 15.8 -> 17.1 mm
- net /GPIO2: track 76.6 -> 77.7 mm
- net /QSPI_SD3: track 17.2 -> 18.2 mm
- net /GPIO29_ADC3: track 29.5 -> 28.5 mm
- net /GPIO15: track 76.5 -> 75.6 mm
- net /GPIO27_ADC1: track 61.9 -> 61.3 mm
- net /GPIO26_ADC0: track 64.9 -> 64.2 mm
- net /GPIO28_ADC2: track 75.8 -> 75.1 mm
- net /GPIO20_TRANS: track 55.6 -> 56.1 mm
- net /GPIO18_TRANS: track 53.4 -> 53.9 mm
- net /GPIO19_TRANS: track 54.2 -> 54.7 mm
